Commit message: Enhance README and URDF for NavProMini integration
- Updated README.md to include the `navpromini_controller` package details, hardware requirements, and launch instructions for real robot workflows.
- Revised wheel radius and track specifications for accuracy.
- Added IMU link and joint definitions in NavProMini.xacro for onboard QMI8658 integration.
- Improved clarity on required interfaces and common failure modes for real robot operations.

File: navpromini_description/urdf/NavProMini.xacro (robot description, xacro)
@@ -252,3 +252,16 @@
     <child link="FC_1"/>
   </joint>
+  <!-- Onboard QMI8658 (Waveshare General Driver); fuse later -->
+  <link name="imu_link">
+    <inertial>
+      <origin xyz="0 0 0" rpy="0 0 0"/>
+      <mass value="0.001"/>
+      <inertia ixx="1e-6" iyy="1e-6" izz="1e-6" ixy="0" iyz="0" ixz="0"/>
+    </inertial>
+  </link>
+  <joint name="imu_joint" type="fixed">
+    <origin xyz="0 0 0.08" rpy="0 0 0"/>
+    <parent link="base_link"/>
+    <child link="imu_link"/>
+  </joint>
 </robot>

Commit message: Refactor odometry parameters and calculations for improved accuracy
- Updated `odom_params.yaml` to align with the diff_drive_controller model, adjusting `wheel_radius`, `wheel_separation`, and `ticks_per_revolution`.
- Enhanced `odom_node.py` to implement the new odometry calculations based on the updated parameters, ensuring accurate movement tracking.
- Improved logging and error handling for odometry consistency checks.
- Revised URDF and XACRO files to reflect the updated wheel specifications for better integration with the odometry system.

File: navpromini_description/urdf/NavProMini.xacro (robot description, xacro)
@@ -7,5 +7,5 @@
   <xacro:property name="motor_effort" value="0.981"/>
   <xacro:property name="motor_velocity" value="31.416"/>
-  <xacro:property name="wheel_radius" value="0.034"/>
+  <xacro:property name="wheel_radius" value="0.0325"/>  <!-- 65 mm diameter -->
   <xacro:property name="wheel_width" value="0.028"/>
   <!-- ROS base_link: +X forward, +Y left. Mass lives here for stable physics. -->

Commit message: Enhance RPLidar launch and configuration for improved functionality
- Added 'inverted' launch argument to the RPLidar launch file to support mirrored scans.
- Updated logging to include the inverted state of the RPLidar for better diagnostics.
- Adjusted URDF to correct the Lidar joint orientation, ensuring accurate scan alignment.
- Modified SLAM and navigation launch files to set 'use_sim_time' to false for real robot operation.
- Improved joystick and keyboard launch configurations to clarify usage and adjust parameters for better control responsiveness.

File: navpromini_description/urdf/NavProMini.xacro (robot description, xacro)
@@ -242,6 +242,9 @@
     <child link="BLC_1"/>
   </joint>
+  <!-- Lidar optical +X must match base_link +X (robot forward).
+       chassis is +90° yaw vs base_link (CAD), so cancel with -90° here.
+       Without this, /scan is 90° off → SLAM smear + wrong motion in RViz. -->
   <joint name="LidarJoint" type="fixed">
-    <origin xyz="0.001341 -0.032462 0.188795" rpy="0 0 0"/>
+    <origin xyz="0.001341 -0.032462 0.188795" rpy="0 0 -1.57079632679"/>
     <parent link="chassis"/>
     <child link="lidar_1"/>

Commit message: Enhance Lidar configuration and integration in launch and URDF files
- Added 'lidar_yaw' launch argument to allow adjustable Lidar orientation for accurate scan alignment.
- Updated NavProMini.xacro to include Lidar pose properties and ensure correct joint orientation relative to the base_link.
- Improved comments for clarity on Lidar positioning and its impact on SLAM performance.

File: navpromini_description/urdf/NavProMini.xacro (robot description, xacro)
@@ -9,4 +9,12 @@
   <xacro:property name="wheel_radius" value="0.0325"/>  <!-- 65 mm diameter -->
   <xacro:property name="wheel_width" value="0.028"/>
+  <!-- Lidar pose in base_link (+X forward). Yaw is tunable at launch:
+       xacro ... lidar_yaw:=±1.5708 if /scan is 90° off vs driving direction. -->
+  <xacro:arg name="lidar_yaw" default="0.0"/>
+  <xacro:property name="lidar_yaw" value="$(arg lidar_yaw)"/>
+  <!-- chassis joint origin (0.001341, -0.032462, 0.188795) rotated by +90° yaw -->
+  <xacro:property name="lidar_x" value="0.032462"/>
+  <xacro:property name="lidar_y" value="0.001341"/>
+  <xacro:property name="lidar_z" value="0.188795"/>
   <!-- ROS base_link: +X forward, +Y left. Mass lives here for stable physics. -->
   <link name="base_link">
@@ -171,6 +179,7 @@
       <inertia ixx="1e-5" iyy="1e-5" izz="2e-05" ixy="0" iyz="0" ixz="0"/>
     </inertial>
-    <visual>
-      <origin xyz="-0.001341 0.032462 -0.188795" rpy="0 0 0"/>
+    <!-- Mesh is CAD/chassis-oriented; rotate +90° so it matches chassis visual. -->
+    <visual>
+      <origin xyz="-0.001341 0.032462 -0.188795" rpy="0 0 1.57079632679"/>
       <geometry>
         <mesh filename="package://navpromini_description/meshes/lidar_1.stl" scale="0.001 0.001 0.001"/>
@@ -179,5 +188,5 @@
     </visual>
     <collision>
-      <origin xyz="-0.001341 0.032462 -0.188795" rpy="0 0 0"/>
+      <origin xyz="-0.001341 0.032462 -0.188795" rpy="0 0 1.57079632679"/>
       <geometry>
         <mesh filename="package://navpromini_description/meshes/lidar_1.stl" scale="0.001 0.001 0.001"/>
@@ -242,10 +251,9 @@
     <child link="BLC_1"/>
   </joint>
-  <!-- Lidar optical +X must match base_link +X (robot forward).
-       chassis is +90° yaw vs base_link (CAD), so cancel with -90° here.
-       Without this, /scan is 90° off → SLAM smear + wrong motion in RViz. -->
+  <!-- Optical frame on base_link (not chassis): scan 0° = base +X = drive forward.
+       Parenting under chassis inherited CAD +90° yaw and smeared SLAM maps. -->
   <joint name="LidarJoint" type="fixed">
-    <origin xyz="0.001341 -0.032462 0.188795" rpy="0 0 -1.57079632679"/>
-    <parent link="chassis"/>
+    <origin xyz="${lidar_x} ${lidar_y} ${lidar_z}" rpy="0 0 ${lidar_yaw}"/>
+    <parent link="base_link"/>
     <child link="lidar_1"/>
   </joint>

Commit message: Enhance multi-robot simulation configuration for NavProMini
- Updated `NavProMini.gazebo` and `NavProMini.xacro` to support multi-robot setups with adjustable topic and frame prefixes, improving compatibility with RMF.
- Increased maximum linear and angular velocities for faster simulation performance while ensuring compliance with fleet limits.
- Adjusted Lidar range settings to enhance obstacle detection capabilities in confined spaces.
- Introduced a new package `navpromini_rmf_sim` for managing multi-robot simulation assets, including launch files and configuration for RMF integration.
- Added comprehensive README documentation for setup and usage instructions, facilitating easier deployment and configuration of the simulation environment.

File: navpromini_description/urdf/NavProMini.xacro (robot description, xacro)
@@ -3,5 +3,4 @@
   <xacro:include filename="$(find navpromini_description)/urdf/materials.xacro" />
   <xacro:include filename="$(find navpromini_description)/urdf/NavProMini.trans" />
-  <xacro:include filename="$(find navpromini_description)/urdf/NavProMini.gazebo" />
   <!-- Motor limits: 10 kg.cm = 0.981 N.m, 300 RPM = 31.416 rad/s -->
   <xacro:property name="motor_effort" value="0.981"/>
@@ -9,8 +8,17 @@
   <xacro:property name="wheel_radius" value="0.0325"/>  <!-- 65 mm diameter -->
   <xacro:property name="wheel_width" value="0.028"/>
+  <!-- Multi-robot Gazebo: launch passes topic_prefix:=/robot1 frame_prefix:=robot1/
+       Single-robot defaults keep absolute /cmd_vel, /odom, /scan. -->
+  <xacro:arg name="robot_namespace" default=""/>
+  <xacro:arg name="topic_prefix" default=""/>
+  <xacro:arg name="frame_prefix" default=""/>
+  <xacro:property name="topic_prefix" value="$(arg topic_prefix)"/>
+  <xacro:property name="frame_prefix" value="$(arg frame_prefix)"/>
   <!-- Lidar pose in base_link (+X forward). Yaw is tunable at launch:
        xacro ... lidar_yaw:=±1.5708 if /scan is 90° off vs driving direction. -->
   <xacro:arg name="lidar_yaw" default="0.0"/>
   <xacro:property name="lidar_yaw" value="$(arg lidar_yaw)"/>
+  <!-- After topic/frame prefix properties so NavProMini.gazebo can use them. -->
+  <xacro:include filename="$(find navpromini_description)/urdf/NavProMini.gazebo" />
   <!-- chassis joint origin (0.001341, -0.032462, 0.188795) rotated by +90° yaw -->
   <xacro:property name="lidar_x" value="0.032462"/>
@@ -22,6 +30,7 @@
       <!-- Between drive wheels (x≈0.067) and rear caster (x≈-0.074) -->
       <origin xyz="0.02 0.0 0.05" rpy="0 0 0"/>
-      <mass value="5.0"/>
-      <inertia ixx="0.04" iyy="0.04" izz="0.05" ixy="0.0" iyz="0.0" ixz="0.0"/>
+      <!-- Half mass for smoother Gazebo multi-robot sim -->
+      <mass value="2.5"/>
+      <inertia ixx="0.02" iyy="0.02" izz="0.025" ixy="0.0" iyz="0.0" ixz="0.0"/>
     </inertial>
   </link>
